Commit message: fix: ydlidar orientation and motor connector

File: urdf/oit_minibot_light_v5.xacro (robot description, xacro)
@@ -26,8 +26,8 @@
   <xacro:property name="laser_w" value="0.06" />
   <xacro:property name="laser_h" value="0.06" />
-  <xacro:property name="laser_x" value="0.05" />
-  <xacro:property name="laser_z" value="0.02" />
+  <xacro:property name="laser_x" value="0.07" />
+  <xacro:property name="laser_z" value="0.0313" />
   <joint name="laser_joint" type="fixed">
-    <origin xyz="${laser_x} 0 ${laser_z}" rpy="${radians(180)} 0 0"/>
+    <origin xyz="${laser_x} 0 ${laser_z}" rpy="0 0 ${radians(-90)}"/>
     <parent link="base_link"/>
     <child link="base_laser_link"/>
